Commit message: [update] Enhanced URDF with detailed servo brackets and hardware specs
Based on procurement list (四足机器恐龙_采购清单.xlsx), added comprehensive
mechanical details to URDF model:

## New Features
- Added 8 bracket links (4× hip_bracket, 4× knee_bracket)
  - Hip brackets: 40×50×20mm aluminum U-brackets for shoulder servo mounting
  - Knee brackets: 30×40×15mm aluminum brackets at upper leg base
  - Visual representation with silver material (0.7, 0.7, 0.75, 1)

- Enhanced header with complete hardware specifications:
  - Body structure: 200×110×36mm (3mm acrylic + 30mm standoffs)
  - DS3218 servo specs: 21 kg·cm torque, 60g weight, 270° range
  - Mounting hardware: 12× U-brackets, 16× MR105ZZ bearings
  - PCA9685 channel allocation table (CH0-11)

- Added detailed joint comments for all 12 joints:
  - Servo model and channel assignment
  - Function description (外展/内收, 前后摆动, 膝盖弯曲)
  - Rotation axis and angle ranges
  - Mounting position and bearing configuration
  - Connection method (M2×8 screws, servo horn)

## Structure Changes
- Total links: 17 → 25 (added 8 bracket links)
- Total joints: 16 → 24 (8 fixed bracket joints)
- All brackets use fixed joints attached to parent links

## Validation
✓ XML syntax validated
✓ All 8 bracket links present
✓ Joint axes verified (hip=X-axis, shoulder/knee=Y-axis)
✓ Coordinate system consistent (X-forward, Y-left, Z-up)

## Purpose
Provides clear mechanical assembly reference for:
- Purchasing correct servo brackets
- Understanding U-bracket mounting structure
- Identifying bearing support positions
- Planning leg-to-body connection assembly

Co-Authored-By: Claude Opus 4 <noreply@anthropic.com>

File: urdf/dino_quadruped.urdf (robot description, URDF)
Before this commit: robot dino_quadruped, 17 links, 16 joints
Links:
- added link fl_hip_bracket, mass 0.05; collision box size=0.02 0.04 0.05; visual box size=0.02 0.04 0.05
- added link fl_knee_bracket, mass 0.03; collision box size=0.015 0.03 0.04; visual box size=0.015 0.03 0.04
- added link fr_hip_bracket, mass 0.05; collision box size=0.02 0.04 0.05; visual box size=0.02 0.04 0.05
- added link fr_knee_bracket, mass 0.03; collision box size=0.015 0.03 0.04; visual box size=0.015 0.03 0.04
- added link rl_hip_bracket, mass 0.05; collision box size=0.02 0.04 0.05; visual box size=0.02 0.04 0.05
- added link rl_knee_bracket, mass 0.03; collision box size=0.015 0.03 0.04; visual box size=0.015 0.03 0.04
- added link rr_hip_bracket, mass 0.05; collision box size=0.02 0.04 0.05; visual box size=0.02 0.04 0.05
- added link rr_knee_bracket, mass 0.03; collision box size=0.015 0.03 0.04; visual box size=0.015 0.03 0.04
Joints:
- added joint fl_hip_bracket_joint: type fixed, parent fl_hip, child fl_hip_bracket, origin xyz=0 0 0 rpy=0 0 0
- added joint fl_knee_bracket_joint: type fixed, parent fl_upper_leg, child fl_knee_bracket, origin xyz=0 0 -0.10 rpy=0 0 0
- added joint fr_hip_bracket_joint: type fixed, parent fr_hip, child fr_hip_bracket, origin xyz=0 0 0 rpy=0 0 0
- added joint fr_knee_bracket_joint: type fixed, parent fr_upper_leg, child fr_knee_bracket, origin xyz=0 0 -0.10 rpy=0 0 0
- added joint rl_hip_bracket_joint: type fixed, parent rl_hip, child rl_hip_bracket, origin xyz=0 0 0 rpy=0 0 0
- added joint rl_knee_bracket_joint: type fixed, parent rl_upper_leg, child rl_knee_bracket, origin xyz=0 0 -0.10 rpy=0 0 0
- added joint rr_hip_bracket_joint: type fixed, parent rr_hip, child rr_hip_bracket, origin xyz=0 0 0 rpy=0 0 0
- added joint rr_knee_bracket_joint: type fixed, parent rr_upper_leg, child rr_knee_bracket, origin xyz=0 0 -0.10 rpy=0 0 0
